File: Untitled.kicad_pcb (KiCad board)
At the start: 2 copper layers, 0 parts

Commit message: ネット幅リストに追記
Other:
- net class Default: via_dia 0.8 -> 0.65; via_drill 0.3 -> 0.35
- net class wire-0.2 added: clearance 0.1524, trace_width 0.2, via_dia 0.6, via_drill 0.3
- net class wire-0.3 added: clearance 0.1524, trace_width 0.3, via_dia 0.6, via_drill 0.3
- net class wire-0.4 added: clearance 0.1524, trace_width 0.4, via_dia 0.6, via_drill 0.3
- net class wire-0.5 added: clearance 0.1524, trace_width 0.5, via_dia 0.6, via_drill 0.3
- net class wire-0.6 added: clearance 0.1524, trace_width 0.6, via_dia 0.6, via_drill 0.3
- net class wire-0.7 added: clearance 0.1524, trace_width 0.7, via_dia 0.7, via_drill 0.4
- net class wire-0.8 added: clearance 0.1524, trace_width 0.8, via_dia 0.8, via_drill 0.5
- net class wire-0.9 added: clearance 0.1524, trace_width 0.9, via_dia 0.9, via_drill 0.6
- net class wire-1.0 added: clearance 0.1524, trace_width 1, via_dia 1, via_drill 0.7
Changed lines of the file:
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@@
     (zone_45_only no)
     (trace_min 0.2)
-    (via_size 0.8)
-    (via_drill 0.3)
+    (via_size 0.65)
+    (via_drill 0.35)
     (via_min_size 0.6)
     (via_min_drill 0.3)
@@
     (clearance 0.1524)
     (trace_width 0.25)
-    (via_dia 0.8)
+    (via_dia 0.65)
+    (via_drill 0.35)
+    (uvia_dia 0.3)
+    (uvia_drill 0.1)
+  )
+  (net_class wire-0.2 ""
+    (clearance 0.1524)
+    (trace_width 0.2)
+    (via_dia 0.6)
     (via_drill 0.3)
     (uvia_dia 0.3)
     (uvia_drill 0.1)
+  )
+  (net_class wire-0.3 ""
+    (clearance 0.1524)
+    (trace_width 0.3)
+    (via_dia 0.6)
+    (via_drill 0.3)
+    (uvia_dia 0.3)
+    (uvia_drill 0.1)
+  )
+  (net_class wire-0.4 ""
+    (clearance 0.1524)
+    (trace_width 0.4)
+    (via_dia 0.6)
+    (via_drill 0.3)
+    (uvia_dia 0.3)
+    (uvia_drill 0.1)
+  )
+  (net_class wire-0.5 ""
+    (clearance 0.1524)
+    (trace_width 0.5)
+    (via_dia 0.6)
+    (via_drill 0.3)
+    (uvia_dia 0.3)
+    (uvia_drill 0.1)
+  )
+  (net_class wire-0.6 ""
+    (clearance 0.1524)
+    (trace_width 0.6)
+    (via_dia 0.6)
+    (via_drill 0.3)
+    (uvia_dia 0.3)
+    (uvia_drill 0.1)
+  )
+  (net_class wire-0.7 ""
+    (clearance 0.1524)
+    (trace_width 0.7)
+    (via_dia 0.7)
+    (via_drill 0.4)
+    (uvia_dia 0.3)
+    (uvia_drill 0.1)
+  )
+  (net_class wire-0.8 ""
+    (clearance 0.1524)
+    (trace_width 0.8)
+    (via_dia 0.8)
+    (via_drill 0.5)
+    (uvia_dia 0.3)
+    (uvia_drill 0.1)
+  )
+  (net_class wire-0.9 ""
+    (clearance 0.1524)
+    (trace_width 0.9)
+    (via_dia 0.9)
+    (via_drill 0.6)
+    (uvia_dia 0.3)
+    (uvia_drill 0.1)
+  )
+  (net_class wire-1.0 ""
+    (clearance 0.1524)
+    (trace_width 1)
+    (via_dia 1)
+    (via_drill 0.7)
+    (uvia_dia 0.3)
+    (uvia_drill 0.1)
